Commit message: feat(go2_description): Velodyne VLP-16 이식 — 유효 점 2181 → 4213
내장 L1 은 머리에 달린 200도·10m 센서다. pipeline 은 야외라 ray 의 79% 가
아무것도 못 맞히고 스캔당 실제 점이 2181개뿐이었다. clearpath_ws 의 Go2 가
쓰는 VLP-16(360도, 131m) 을 같은 스펙으로 옮겼다 — 그래야 두 스택의 매핑
결과를 같은 센서 기준으로 비교할 수 있다.

    센서        스캔당 유효 점   inf 비율   RTF
    L1           2181            79%       1.00
    VLP-16       4213            40%       1.00

velodyne:=true 로 켠다. 둘 중 하나만 뜨고(L1 은 xacro:unless 로 빠진다)
**토픽이 `scan` 으로 같아서** 브리지·/scan/points 소비자·lidar_time_relay 가
그대로 동작한다. 바뀌는 건 frame_id 뿐이고(velodyne), TF 는 고정 조인트라
robot_state_publisher 가 낸다.

형상은 VLP16_*.dae 대신 단순 원통이다. 그 메시는 clearpath_ws 에 있어서
가져오면 두 워크스페이스가 묶인다. 시뮬에 필요한 건 충돌·관성과 센서 원점
이고 비주얼은 장식이다.

장착은 trunk 위 0.10m 수평. clearpath_ws 는 base_link 기준 (0.2, 0, 0.08)
인데 이 스택은 몸통 원점이 달라서 높이만 맞췄다. 앞으로 치우치면 360도
스캔이 몸통에 가린다.

File: descriptions/unitree/go2_description/xacro/gazebo.xacro (robot description, xacro)
@@ -268,4 +268,5 @@
     </gazebo>
     </xacro:unless>
+    <xacro:unless value="$(arg VELODYNE)">
     <gazebo reference="lidar">
       <sensor name='L1_lidar' type='gpu_lidar'>
@@ -298,4 +299,10 @@
       </sensor>
     </gazebo>
+    </xacro:unless>
+    <!-- 같은 `scan` 토픽으로 낸다. 둘 중 하나만 켜지므로 겹치지 않고,
+         브리지와 /scan/points 소비자들은 그대로 쓸 수 있다. -->
+    <xacro:if value="$(arg VELODYNE)">
+      <xacro:velodyne_vlp16_gazebo topic="scan"/>
+    </xacro:if>
   </xacro:if>
 </robot>

File: descriptions/unitree/go2_description/xacro/robot.xacro (robot description, xacro)
@@ -4,7 +4,10 @@
   <xacro:arg name="GAZEBO" default="false"/>
   <xacro:arg name="CLASSIC" default="false"/>
+  <!-- Velodyne VLP-16 instead of the built-in L1 head lidar. See velodyne.xacro. -->
+  <xacro:arg name="VELODYNE" default="false"/>
   <xacro:include filename="$(find go2_description)/xacro/const.xacro"/>
   <xacro:include filename="$(find go2_description)/xacro/materials.xacro"/>
   <xacro:include filename="$(find go2_description)/xacro/leg.xacro"/>
+  <xacro:include filename="$(find go2_description)/xacro/velodyne.xacro"/>
   <xacro:if value="$(arg GAZEBO)">
     <xacro:if value="$(arg CLASSIC)">
@@ -125,4 +128,12 @@
   <link name="lidar">
   </link>
+  <!-- 몸통 위, 수평. 360도 스캔이 몸통에 가리지 않도록 위로 올린다.
+       (clearpath_ws 는 base_link 기준 0.2 0 0.08 인데, 그쪽은 몸통 원점이
+        달라서 높이만 맞춰 옮겼다.) -->
+  <xacro:if value="$(arg VELODYNE)">
+    <xacro:velodyne_vlp16 parent="trunk">
+      <origin rpy="0 0 0" xyz="0.0 0 0.10"/>
+    </xacro:velodyne_vlp16>
+  </xacro:if>
   <xacro:leg name="FR" mirror="-1" mirror_dae="False" front_hind="1" front_hind_dae="True"/>
   <xacro:leg name="FL" mirror="1" mirror_dae="True" front_hind="1" front_hind_dae="True"/>
